File: Power_Amplifier/Discrete_Channel.sch (KiCad schematic (older format))
At the start: 68 parts, among them J1 Conn_01x05_Male, J2 Conn_01x06_Male, J3 Conn_01x05_Male, J4 Banna Jack, U1 TPA3244, U2 LM4562

Commit message: WiP - Schematic Edits
Fixed Zobel Network
Adopted TPA3245

TODO: Revise PCB
Parts:
- added R? (x2): 2.7k, Resistor_SMD:R_0805_2012Metric_Pad1.20x1.40mm_HandSolder, symbol Device:R_Small_US
- L2: footprint Inductor_SMD:L_12x12mm_H6mm -> (none); Note https://www.digikey.com/en/products/detail/w%C3%BCrth-elektronik/74477110/1638613 -> https://www.digikey.com/en/products/detail/w%C3%BCrth-elektronik/7443631000/2440338; Part 74477110 -> 7443631000
- U1: value TPA3244 -> TPA3245; symbol Discrete_Channel-rescue:TPA3244-TPA3244 -> TPA3244:TPA3245
Connections:
- net DVDD: now also U1.11 (DVDD), U1.4 (M2); no longer U1.12 (DVDD), U1.19 (M2)
- net FB_A: now also R?.1; no longer C19.2, R8.1, U2.1
- net FB_B: now also R?.1; no longer C18.2, R7.1, U2.7
- net GND: now also U1.12 (GND), U1.13 (GND), U1.3 (M1); no longer U1.10 (GND), U1.11 (GND), U1.20 (M1)
- net GNDA: now also U1.16 (INPUT_C), U1.17 (INPUT_D); no longer U1.6 (INPUT_D), U1.7 (INPUT_C)
- net OSC_IOM: now also U1.9 (OSC_IOM); no longer U1.14 (OSC_IOM)
- net OSC_IOP: now also U1.10 (OSC_IOP); no longer U1.13 (OSC_IOP)
- net OUT_A: now also U1.39 (OUT_A), U1.40 (OUT_A); no longer U1.27 (OUT_A), U1.28 (OUT_A)
- net OUT_B: now also U1.35 (OUT_B); no longer U1.32 (OUT_B)
- net OUT_C: now also U1.32 (OUT_C); no longer U1.35 (OUT_C)
- net OUT_D: now also U1.27 (OUT_D), U1.28 (OUT_D); no longer U1.39 (OUT_D), U1.40 (OUT_D)
- net ~ERROR: now also U1.21 (~CLIP_OTP); no longer U1.2 (~CLIP_OTP)
- net ~FAULT: now also U1.19 (~FAULT); no longer U1.4 (~FAULT)
- net ~RESET: now also U1.18 (~RESET); no longer U1.5 (~RESET)
- net at C8.2, R2.1: now also U1.22 (GVDD_CD); no longer U1.1 (GVDD_CD)
- net at C14.2, L1.1: now also U1.2 (VDD); no longer U1.21 (VDD)
- net at C6.2, R1.1: now also U1.1 (GVDD_AB); no longer U1.22 (GVDD_AB)
- net at C15.2: now also U1.20 (VBG); no longer U1.3 (VBG)
- net at C16.2: now also U1.14 (AVDD); no longer U1.9 (AVDD)
- net at JP1.2, R3.2: now also U1.8 (FREQ_ADJ); no longer U1.15 (FREQ_ADJ)
- net at R4.2: now also U1.7 (OC_ADJ); no longer U1.16 (OC_ADJ)
- net at C9.1: now also U1.15 (C_START); no longer U1.8 (C_START)
- net at C21.1: now also U1.6 (INPUT_B); no longer U1.17 (INPUT_B)
- net at C20.1: now also U1.5 (INPUT_A); no longer U1.18 (INPUT_A)
- net at C22.1: now also U1.44 (BST_A); no longer U1.23 (BST_A)
- net at C23.1: now also U1.43 (BST_B); no longer U1.24 (BST_B)
- net at C24.1: now also U1.24 (BST_C); no longer U1.43 (BST_C)
- net at C25.1: now also U1.23 (BST_D); no longer U1.44 (BST_D)
- new net: C19.2, R8.1, R?.2, U2.1
- new net: C18.2, R7.1, R?.2, U2.7
Other:
- note added: "(Optional) Post-Filter Feedback Implemented\nBased on (Figure 2; Table 1) of Ti's SLAA788A"
- note added: "3"
- note added: "Note: L1 based on design of\nTPA3244EVM Evaluation Module"
- note added: "Note: R3 Sets F_PWM to 450 kHz per (7.3)"
- note added: "Revision Notes:\nAdopted TPA3245 for Heatsinking"
- note added: "TPA3245\n(PBTL) Outputs Paralleled afted LC Filter"
- note removed: "TPA3244\nOutputs Paralleled afted LC Filter"
- moved on the sheet: C10, C11, C12, C13, C18, C19, JP2, R5, R6, R7, R8, U2A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
